File: Hardware/ESP32_BLDC_Motor_Driver.sch (EAGLE design)
At the start: 16 parts, among them U1 TMC6300

Commit message: Updates to schematic, added new part
Continued work with schematic, added more parts to the project/library (TMC6300, output connector for motor, ESP32)
Parts:
- added J1: (no value), SparkFun-Connectors:USB_C_4-LAYER_PADS
- added J2: 0532610371, 0532610371:0532610371
- added J3: POWER_JACKPOWER_JACK_SLOT, SparkFun-Connectors:POWER_JACKPOWER_JACK_SLOT
- added LOGO1: SFE_LOGO_NAME.5_INCH, SparkFun-Aesthetics:SFE_LOGO_NAME.5_INCH
- added LOGO2: OSHW-LOGOM, SparkFun-Aesthetics:OSHW-LOGOM
- added LOGO3: SFE_LOGO_FLAME.5_INCH, SparkFun-Aesthetics:SFE_LOGO_FLAME.5_INCH
- added U2: CH340G, SparkFun-IC-Comms:CH340GSMD
Connections:
- new net N$2: J2.1, U1.W
- new net N$7: J2.2, U1.V
- new net N$8: J2.3, U1.U
Other:
- note added: "Connectors"
- moved on the sheet: C1, C2, C3, C4, R1

Commit message: Added datasheet, further schematic work
Added datasheet for an IC and continued work on schematic. All sections should now be on the project, need to be checked and completed.
Parts:
- added BYP: JUMPER-SMT_2_NO_SILK, SparkFun-Jumpers:JUMPER-SMT_2_NO_SILK
- added C10, C9: 10pF, SparkFun-Capacitors:10PF-0603-50V-5%
- added C11: 100pF, SparkFun-Capacitors:100PF-0603-50V-5%
- added C12, C13, C14, C15, C7: 0.1uF, SparkFun-Capacitors:0.1UF-0603-25V-5%
- added C16, C18: 10uF, SparkFun-Capacitors:10UF-0603-6.3V-20%
- added C17: 1.0uF, SparkFun-Capacitors:1.0UF-0603-16V-10%-X7R
- added C19, C8: 0.1uF, SparkFun-Capacitors:0.1UF-0603-25V-10%-X7R-WE
- added C5: 47uF, SparkFun-Capacitors:47UF-POLAR-PANASONIC_D-35V-20%
- added C6: 10uF, SparkFun-Capacitors:10UF-POLAR-EIA3216-16V-10%(TANT)
- added D, PWR, S: JUMPER-SMT_2_NC_TRACE_SILK, SparkFun-Jumpers:JUMPER-SMT_2_NC_TRACE_SILK
- added D1: 1A/40V/500mV, SparkFun-DiscreteSemi:DIODE-SCHOTTKY-SS14
- added D2: YELLOW, SparkFun-LED:LED-YELLOW0603
- added D3, D5: GREEN, SparkFun-LED:LED-GREEN0603
- added D4: BLUE, SparkFun-LED:LED-BLUE0603
- added D6: RED, SparkFun-LED:LED-RED0603
- added F1: 6V/2A, SparkFun-Fuses:PPTC_6V2A
- added Q1: 20V/4.2A/52mΩ/1.4W, SparkFun-DiscreteSemi:MOSFET_PCH-DMG2305UX-7
- added R10, R11, R12, R7, R8, R9: 100k, SparkFun-Resistors:100KOHM-0603-1/10W-1%
- added R13, R3: 2.2k, SparkFun-Resistors:2.2KOHM-0603-1/10W-1%
- added R14: 0.012ohm, SparkFun-Resistors:0.012OHM0603
- added R15, R2: 330, SparkFun-Resistors:330OHM-0603-1/10W-1%
- added R16: 1k, SparkFun-Resistors:1KOHM-0603-1/10W-1%
- added R17, R4: 10k, SparkFun-Resistors:10KOHM-0603-1/10W-1%
- added R5: 390, SparkFun-Resistors:390OHM-0603-1/10W-1%
- added R6: 240, SparkFun-Resistors:240OHM-0603-1/10W-1%
- added S1: MOMENTARY-SWITCH-SPST-SMD-4.6X2.8MM, SparkFun-Switches:MOMENTARY-SWITCH-SPST-SMD-4.6X2.8MM
- added U3: LM1117, SparkFun-IC-Power:V_REG_LM1117SOT223
- added Y1: 12MHz, SparkFun-Clocks:CRYSTAL-12MHZ
Connections:
- removed net EN: U$1.(GPIO15/ADC2:3/TOUCH3/RTC13/SPICSO/U0RTS)MTDO
- new net !DTR!: U2.!DTR
- new net D+: J1.D+, U2.UD+
- new net D-: J1.D-, U2.UD-
- new net N$15: C5.-
- new net N$16: D1.A, J3.PWR
- new net N$17: BYP.1, F1.1, J1.VBUS
- new net N$18: D3.A, R2.1
- new net N$19: D2.A, R3.1
- new net N$20: J3.GND, Q1.G, R4.1
- new net N$21: C5.+, D1.C, U3.IN
- new net N$22: R5.2, R6.1, U3.ADJ
- new net N$23: PWR.1, R16.2
- new net N$24: S.2, U1.VIO/!STDBY!
- new net N$25: C9.2, U2.XI, Y1.2
- new net N$26: C10.2, U2.XO, Y1.1
- new net N$27: C10.1, C9.1
- new net N$28: D4.A, S.1
- new net N$29: D4.C, R13.2
- new net N$30: C8.1, U1.1.8VOUT
- new net N$31: D.2, U1.DIAG
- new net N$32: D.1, D5.A
- new net N$33: D5.C, R15.2
- new net N$34: D6.A, R16.1
- new net RX-I: D2.C, U2.TXO
- new net SENSE: R14.2, U$1.(GPIO15/ADC2:3/TOUCH3/RTC13/SPICSO/U0RTS)MTDO, U1.BRUV, U1.BRW
- new net SHLD: J1.SHLD
- new net TX-O: D3.C, U2.RXI
- new net USBVCC: BYP.2, F1.2, Q1.D
- net 3.3V: now also C11.1, C12.1, C13.1, C14.1, C15.1, C16.1, C17.1, C18.1, C19.1, C6.+, C7.1, PWR.2, Q1.S, R17.2, R2.2, R3.2, R4.2, R6.2, U1.VS, U2.V3, U2.VCC, U3.OUT
- net CHIP_PU: now also R17.1, S1.2
- net GND: now also C11.2, C12.2, C13.2, C14.2, C15.2, C16.2, C17.2, C18.2, C19.2, C6.-, C7.2, C8.2, D6.C, J1.GND, J3.GNDBREAK, R10.1, R11.1, R12.1, R13.1, R14.1, R15.1, R5.1, R7.1, R8.1, R9.1, S1.1, U1.GND, U2.GND
- net UH: now also R12.2, U1.UH
- net UL: now also R11.2, U1.UL
- net VH: now also R10.2, U1.VH
- net VL: now also R9.2, U1.VL
- net WH: now also R8.2, U1.WH
- net WL: now also R7.2, U1.WL
Other:
- note added: "1"
- note added: "19"
- note added: "26"
- note added: "3, 4"
- note added: "37"
- note added: "46, 43"
- note added: "Cut Jumper D to disable diagnostic LED"
- note added: "Cut Jumper PWR to disable Power LED"
- note added: "Cut Jumper S to disable standby LED"
- note added: "Near VDDA"
- note added: "Near VDDA3P3"
- note added: "Near VDDA_LNA"
- note added: "Near VDDPST_CPU"
- note added: "Near VDDPST_RTC"
- note added: "Near VDDPST_SDIO"
- note added: "Power LED"
- note added: "Power Supply"
- note added: "RESET"
- note added: "Reset"
- note added: "USB-to-Serial Converter"
- note added: "Vin Range:"
- note removed: "Connectors"
- moved on the sheet: C1, C2, C3, C4, J1, J2, J3, R1, U1, U2

Commit message: Design updates
Committing updates from the day - need much much more work
Parts:
- removed U3: LM1117, SparkFun-IC-Power:V_REG_LM1117SOT223
- added C20, C21: 22uF, SparkFun-Capacitors:22UF-0603-6.3V-20%
- added C22, C23: 15pF, SparkFun-Capacitors:15PF-0603-50V-5%
- added C24, C25: 10pF, SparkFun-Capacitors:10PF-0603-50V-5%
- added D7: 3.3V, SparkFun-DiscreteSemi:DIODE-ZENER-MM3Z3V3T1G
- added L1: 4.7μH, SparkFun-Coils:4.7μH_SHIELDED_INDUCTORNPIS_LS
- added Q2: 5.8A/30V/35mΩ, SparkFun-DiscreteSemi:MOSFET-NCH-AO3404A
- added U6: AP63357, SparkFun-IC-Power:AP63357
- added Y2: 32.768kHz, SparkFun-Clocks:CRYSTAL-32.768KHZSMD-3.2X1.5
- added Y3: CRYSTAL-26MHZSMD-3.2X2.5, SparkFun-Clocks:CRYSTAL-26MHZSMD-3.2X2.5
- C5: value 47uF -> 0.1uF; device SparkFun-Capacitors:47UF-POLAR-PANASONIC_D-35V-20% -> SparkFun-Capacitors:0.1UF-0603-25V-(+80/-20%)
- C6: value 10uF -> 33pF; device SparkFun-Capacitors:10UF-POLAR-EIA3216-16V-10%(TANT) -> SparkFun-Capacitors:33PF-0603-50V-5%
- C7: value 0.1uF -> 10uF; device SparkFun-Capacitors:0.1UF-0603-25V-5% -> SparkFun-Capacitors:10UF-0603-6.3V-20%
- R5: value 390 -> 93.1k; device SparkFun-Resistors:390OHM-0603-1/10W-1% -> SparkFun-Resistors:93.1KOHM
- R6: value 240 -> 30.1k; device SparkFun-Resistors:240OHM-0603-1/10W-1% -> SparkFun-Resistors:30.1KOHM-0603-1/10W-1%
Connections:
- net N$5 renamed 32K_XP
- net N$6 renamed 32K_XN
- removed net N$15: C5.-
- new net N$36: C6.2, R5.1, R6.2, U6.FB
- new net N$5: C23.1, Y2.2
- new net VIN: C7.1, D1.C, Q1.D, U6.EN, U6.VIN
- net 3.3V: now also C20.1, C21.1, C6.1, D7.C, L1.2, R5.2; no longer C6.+, C7.1, Q1.S, R4.2, R6.2, U3.OUT
- net GND: now also C20.2, C21.2, C22.2, C23.2, C24.1, C25.1, D7.A, R6.1, U6.COMP, U6.GND, Y3.GND; no longer C6.-, R5.1
- net N$1: now also C22.1, Y2.1; no longer U$1.LNA_IN
- net N$21: now also C5.1, U6.BST; no longer C5.+, D1.C, U3.IN
- net N$22: now also C5.2, L1.1, U6.SW; no longer R5.2, R6.1, U3.ADJ
- net N$3: now also C24.2, Y3.1
- net N$4: now also C25.2, Y3.2
- net USBVCC: now also Q1.S, R4.2; no longer Q1.D
Other:
- note added: "26MHz"
- note added: "32.768kHz RTC Crystal"
- moved on the sheet: BYP, C1, C10, C11, C12, C13, C14, C15, C16, C17, C18, C19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

Commit message: Design updates and addition of datasheet
Added datasheet for new IC on board, continued with design
Parts:
- removed C10, C24, C25, C9: 10pF, SparkFun-Capacitors:10PF-0603-50V-5%
- removed C11: 100pF, SparkFun-Capacitors:100PF-0603-50V-5%
- removed C12, C13, C14, C15: 0.1uF, SparkFun-Capacitors:0.1UF-0603-25V-5%
- removed C16: 10uF, SparkFun-Capacitors:10UF-0603-6.3V-20%
- removed C17: 1.0uF, SparkFun-Capacitors:1.0UF-0603-16V-10%-X7R
- removed C22, C23: 15pF, SparkFun-Capacitors:15PF-0603-50V-5%
- removed C3: 10nF, SparkFun-Capacitors:10NF-0603-50V-10%
- removed C4: 3.0nF, SparkFun-Capacitors:3.0NF-0603-50V-5%
- removed Q2: 5.8A/30V/35mΩ, SparkFun-DiscreteSemi:MOSFET-NCH-AO3404A
- removed U$1: ESP32, esp32-thing-temp:ESP32
- removed U2: CH340G, SparkFun-IC-Comms:CH340GSMD
- removed Y1: 12MHz, SparkFun-Clocks:CRYSTAL-12MHZ
- removed Y2: 32.768kHz, SparkFun-Clocks:CRYSTAL-32.768KHZSMD-3.2X1.5
- removed Y3: CRYSTAL-26MHZSMD-3.2X2.5, SparkFun-Clocks:CRYSTAL-26MHZSMD-3.2X2.5
- added R18, R19: 5.1k, SparkFun-Resistors:5.1KOHM5.1KOHM-0603-1/10W-1%
- added SHLD: JUMPER-SMT_2_NC_TRACE_SILK, SparkFun-Jumpers:JUMPER-SMT_2_NC_TRACE_SILK
- added U3: ESP-WROOM-3232D-NARROW, SparkFun-RF:ESP-WROOM-3232D-NARROW
- added U4: CH340E_MSOP10, SparkFun-IC-Comms:CH340E_MSOP10
- C1, C2: value 270PF -> 0.1uF; device SparkFun-Capacitors:270PF-0603-50V-5% -> SparkFun-Capacitors:0.1UF-0603-25V-10%-X7R-WE
- R1: value 20k -> 10k; device SparkFun-Resistors:20KOHM-0603-1/10W-1% -> SparkFun-Resistors:10KOHM-0603-1/10W-1%
Connections:
- net USBVCC renamed V_USB
- removed net !DTR!: U2.!DTR
- removed net 0: U$1.(ADC2:1/TOUCH1/RTC11/CLK_OUT1)GPIO0
- removed net 10: U$1.(GPIO10/SPIWP/HS1_DATA3/U1TX)SD_DATA3
- removed net 11: U$1.(GPIO11/SPICSO/HS1_CMD/U1RTS)SD_CMD
- removed net 16: U$1.(HS1_DATA4)GPIO16
- removed net 17: U$1.(HS1_DATA5)GPIO17
- removed net 18: U$1.(VSPICLK/HS1_DATA7)GPIO18
- removed net 19: U$1.(VSPIQ/HS2_DATA2)GPIO19
- removed net 2: U$1.(ADC2:2/TOUCH2/RTC12/SPIWP)GPIO2
- removed net 20: U$1.(VSPID/HS2_DATA3)GPIO20
- removed net 21: U$1.(VSPIHD/HS2_CMD)GPIO21
- removed net 22: U$1.(VSPIWP/HS2_CLK)GPIO22
- removed net 25: U$1.GPIO23
- removed net 32K_XN: U$1.32K_XN(GPIO33/ADC1:5/TOUCH8/RTC8)
- removed net 32K_XP: U$1.32K_XP(GPIO32/ADC1:4/TOUCH9/RTC9)
- removed net 34: U$1.VDET_1(GPI34/ADC1:6)
- removed net 35: U$1.VDET_2(GPI35/ADC1:7)
- removed net 4: U$1.(ADC2:0/TOUCH0/RTC10/SPIHD)GPIO4
- removed net 5: U$1.(VSPICS0/HS1_DATA6)GPIO5
- removed net 6: U$1.(GPIO6/SPICLK/HS1_CLK/U1CTS)SD_CLK
- removed net 7: U$1.(GPIO7/SPI1/HS1_DATA0)SD_DATA0
- removed net 8: U$1.(GPIO8/SPID/HS1_DATA1)SD_DATA1
- removed net 9: U$1.(GPIO9/SPIHD/HS1_DATA2/U1RX)SD_DATA2
- removed net CHIP_PU: R17.1, S1.2, U$1.CHIP_PU
- removed net N$10: C1.1, U$1.SENSOR_CAPP(GPI37/ADC1:1/RTC1)
- removed net N$11: C2.1, U$1.SENSOR_CAPN(GPI38/ADC1:2/RTC2)
- removed net N$12: C2.2, U$1.SENSOR_VN(GPI39/ADC1:3/RTC3)
- removed net N$13: C3.1, C4.1, R1.1, U$1.CAP_10N
- removed net N$14: C4.2, R1.2, U$1.RES_14K
- removed net N$25: C9.2, U2.XI, Y1.2
- removed net N$26: C10.2, U2.XO, Y1.1
- removed net N$27: C10.1, C9.1
- removed net N$5 (its old number): C23.1, Y2.2
- removed net N$9: C1.2, U$1.SENSOR_VP(GPI36/ADC1:0/RTC0)
- removed net UORXD: U$1.(GPIO3/CLK_OUT2/HS2_DATA0)U0RXD
- removed net UOTXD: U$1.(GPIO1/CLK_OUT3/HS2_DATA1)U0TXD
- new net EN: U3.XTAL_P/IOA32
- new net ESP_0: U3.IOA0
- new net ESP_13: U3.PICO2/IOA13
- new net ESP_15: U3.CS2/IOA15
- new net ESP_16: U3.IO16
- new net ESP_17: U3.IO17
- new net ESP_18: U3.SCK3/IO18
- new net ESP_2: U3.IOA2
- new net ESP_34: U3.IA34
- new net ESP_35: U3.IA35
- new net ESP_36: U3.SENSOR_VP/IA36
- new net ESP_39: U3.SENSOR_VN/IA39
- new net ESP_4: U3.IOA4
- new net ESP_5: U3.CS3/IO5
- new net PICO: U3.PICO3/IO23
- new net POCI: U3.POCI3/IO19
- new net RESET: R1.1, R17.1, S1.2, U3.EN
- new net SCL: U3.SCL/IO22
- new net SDA: U3.SDA/IO21
- net 3.3V: now also C1.1, C2.1, R1.2, U3.3V3, U4.V3, U4.VCC; no longer C11.1, C12.1, C13.1, C14.1, C15.1, C16.1, C17.1, U$1.VDD3P3_CPU, U$1.VDD3P3_RTC, U$1.VDDA, U$1.VDDA3P3, U2.V3, U2.VCC
- net D+: now also U4.UD+; no longer U2.UD+
- net D-: now also U4.UD-; no longer U2.UD-
- net GND: now also C1.2, R18.1, R19.1, SHLD.1, U3.GND, U4.GND; no longer C11.2, C12.2, C13.2, C14.2, C15.2, C16.2, C17.2, C22.2, C23.2, C24.1, C25.1, C3.2, U$1.GND, U2.GND, Y3.GND
- net N$1: now also J1.CC1, R19.2; no longer C22.1, Y2.1
- net N$3: now also J1.CC2, R18.2; no longer C24.2, U$1.XTAL_P, Y3.1
- net N$4: now also C2.2, U1.VCP; no longer C25.2, U$1.XTAL_N, Y3.2
- net RX-I: now also D3.C, U3.TX-IO1, U4.RXI; no longer D2.C, U2.TXO
- net SENSE: no longer U$1.(GPIO15/ADC2:3/TOUCH3/RTC13/SPICSO/U0RTS)MTDO
- net SHLD: now also SHLD.2
- net TX-O: now also D2.C, U3.RX-IO3, U4.TXO; no longer D3.C, U2.RXI
- net UH: now also U3.POCI2/IOA12; no longer U$1.(DAC1/ADC2:8/RTC6)GPIO25
- net UL: now also U3.SCK2/IOA14; no longer U$1.(DAC2/ADC2:9/RTC7)GPIO26
- net VH: now also U3.IOA27; no longer U$1.(ADC2:7/TOUCH7/RTC17)GPIO27
- net VL: now also U3.DAC2/IOA26; no longer U$1.(GPIO14/ADC2:6/TOUCH6/RTC16/SPICLK)MTMS
- net WH: now also U3.DAC1/IOA25; no longer U$1.(GPIO12/ADC2:5/TOUCH5/RTC15/SPIQ)MTDI
- net WL: now also U3.XTAL_N/IOA33; no longer U$1.(GPIO13/ADC2:4/TOUCH4/RTC14/SPID/U0CTS)MTCK
Other:
- note removed: "1"
- note removed: "19"
- note removed: "26"
- note removed: "26MHz"
- note removed: "3, 4"
- note removed: "32.768kHz RTC Crystal"
- note removed: "37"
- note removed: "46, 43"
- note removed: "CHIP_PU is the ESP32's enable/reset pin. It must be pulled high to turn the ESP32 on."
- note removed: "Near VDDA"
- note removed: "Near VDDA3P3"
- note removed: "Near VDDA_LNA"
- note removed: "Near VDDPST_CPU"
- note removed: "Near VDDPST_RTC"
- note removed: "Near VDDPST_SDIO"
- moved on the sheet: BYP, C1, C2, D2, D3, Q1, R1, R2, R3, R4

Commit message: Added correct datasheet, continued design
Continued with design of board, nearing finish of schematic design
Parts:
- added J4, J5: (no value), SparkFun-Connectors:CONN_08"
Connections:
- removed net EN: U3.XTAL_P/IOA32
- removed net ESP_4: U3.IOA4
- removed net N$31: D.2, U1.DIAG
- removed net PICO: U3.PICO3/IO23
- removed net POCI: U3.POCI3/IO19
- removed net SCL: U3.SCL/IO22
- removed net SDA: U3.SDA/IO21
- new net DIAG: D.2, U1.DIAG, U3.IOA4
- new net ESP_19: J5.5, U3.POCI3/IO19
- new net ESP_21: J5.6, U3.SDA/IO21
- new net ESP_22: J5.7, U3.SCL/IO22
- new net ESP_23: J5.8, U3.PICO3/IO23
- net 3.3V: now also R4.2
- net ESP_0: now also J4.7
- net ESP_13: now also J4.5
- net ESP_15: now also J4.6
- net ESP_16: now also J5.1
- net ESP_17: now also J5.2
- net ESP_18: now also J5.4
- net ESP_2: now also J4.8
- net ESP_34: now also J4.3
- net ESP_35: now also J4.4
- net ESP_36: now also J4.1
- net ESP_39: now also J4.2
- net ESP_5: now also J5.3
- net SENSE: now also U3.XTAL_P/IOA32
- net V_USB: no longer R4.2
Other:
- note added: "Pin Headers"
- note added: "Vin Range: 6V - 15V"
- note removed: "Vin Range:"
- moved on the sheet: BYP, C1, C18, C19, C2, C20, C21, C5, C6, C7, C8, D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

Commit message: Schematic ready for review
The schematic has been looked over and is ready for review before starting on the layout. Added Sparkle part number to new library component, added datasheet for new component on board
Parts:
- removed D2: YELLOW, SparkFun-LED:LED-YELLOW0603
- removed D3: GREEN, SparkFun-LED:LED-GREEN0603
- removed D6: RED, SparkFun-LED:LED-RED0603
- removed R1: 10k, SparkFun-Resistors:10KOHM-0603-1/10W-1%
- removed R2: 330, SparkFun-Resistors:330OHM-0603-1/10W-1%
- removed R3: 2.2k, SparkFun-Resistors:2.2KOHM-0603-1/10W-1%
- added C3: 0.1uF, SparkFun-Capacitors:0.1UF-0603-25V-10%-X7R-WE
- added D8: RED, SparkFun-LED:LED-RED_0603-KB
- added R20: 2.0k, SparkFun-Resistors:2.0KOHM-0603-1/10W-5%
- added R25: 18k, SparkFun-Resistors:18KOHM
- added U2: OPA344, SparkFun-IC-Amplifiers:OPA344
- FD1, FD2, FD3, FD4: value FIDUCIAL1X2 -> FIDUCIALUFIDUCIAL; device SparkFun-Aesthetics:FIDUCIAL1X2 -> SparkFun-Aesthetics:FIDUCIALUFIDUCIAL
Connections:
- removed net N$18: D3.A, R2.1
- removed net N$19: D2.A, R3.1
- removed net RX-I: D3.C, U3.TX-IO1, U4.RXI
- removed net TX-O: D2.C, U3.RX-IO3, U4.TXO
- new net CH340-RX: U3.TX-IO1, U4.RXI
- new net CH340-TX: U3.RX-IO3, U4.TXO
- new net CURR_SENSE: R25.2, U2G1.OUT, U3.XTAL_P/IOA32
- new net N$6: R20.2, R25.1, U2G1.-IN
- new net SENSE-: R14.1
- net 3.3V: now also C3.1, U2G2.P$V+; no longer R1.2, R2.2, R3.2
- net GND: now also C3.2, D8.C, R20.1, U2G2.P$V-; no longer D6.C, R14.1
- net N$34: now also D8.A; no longer D6.A
- net RESET: no longer R1.1
- net SENSE: now also U2G1.+IN; no longer U3.XTAL_P/IOA32
- net VIN: now also Q1.S; no longer Q1.D
- net V_USB: now also Q1.D; no longer Q1.S
Other:
- moved on the sheet: C1, C18, C19, C2, C8, D, D4, D5, D7, J2, Q1, R10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

Commit message: Design Updates
Created new board file, added output connector to motor output in case users want to use a different motor for this board
Parts:
- removed R16: 1k, SparkFun-Resistors:1KOHM-0603-1/10W-1%
- added C4: 1nF, SparkFun-Capacitors:1.0NF/1000PF-0603-50V-10%
- added J6: 0.1in header, SparkFun-Connectors:CONN_03
- added R1: 4.7k, SparkFun-Resistors:4.7KOHM-0603-1/10W-1%
Connections:
- removed net N$2: J2.1, U1.W
- removed net N$7: J2.2, U1.V
- removed net N$8: J2.3, U1.U
- removed net SENSE-: R14.1
- new net U: J2.1, J6.1, U1.U
- new net V: J2.2, J6.2, U1.V
- new net W: J2.3, J6.3, U1.W
- net GND: now also C4.2, R14.1
- net N$23: now also R1.2; no longer R16.2
- net N$34: now also R1.1; no longer R16.1
- net RESET: now also C4.1
Other:
- moved on the sheet: J2, R17

Commit message: Design Review Updates
Organized file folders, updates from design review - see document for full list of changes. Still needs a little more work before starting fully on the board file
Parts:
- removed R25: 18k, SparkFun-Resistors:18KOHM
- added C10, C11: 22uF, SparkFun-Capacitors:22UF-0603-6.3V-20%
- added C12: 10uF, SparkFun-Capacitors:10UF-0603-6.3V-20%
- added C9: 0.1uF, SparkFun-Capacitors:0.1UF-0603-25V-5%
- added D2: WS2812_2020, SparkFun-LED:WS2812_2020
- added FRAME2: FRAME-LETTER, SparkFun-Aesthetics:FRAME-LETTER
- added J7: QWIIC_RIGHT_ANGLE, SparkFun-Connectors:QWIIC_CONNECTORJS-1MM
- added J8: (no value), SparkFun-Connectors:CONN_02
- added L2: 4.7μH_SHIELDED_INDUCTOR, SparkFun-Coils:4.7μH_SHIELDED_INDUCTOR
- added LOGO4: QWIIC_LOGO_3MM, SparkFun-Aesthetics:QWIIC_LOGO_3MM
- added Q2: (no value), SparkFun-DiscreteSemi:TRANS_NPN_DUAL-MBT3904DW1T1
- added R16, R2, R3: 10k, SparkFun-Resistors:10KOHM-0603-1/10W-1%
- added R21: 20k, SparkFun-Resistors:20KOHM-0603-1/10W-1%
- added R22, R23: 100k, SparkFun-Resistors:100KOHM-0603-1/10W-1%
- added S2, S3, S4: MOMENTARY-SWITCH-SPST-SMD-4.6X2.8MM, SparkFun-Switches:MOMENTARY-SWITCH-SPST-SMD-4.6X2.8MM
- added TP1, TP10, TP11, TP2, TP3, TP4, TP5, TP6, TP7, TP8, TP9: TEST-POINT3X4, SparkFun-Connectors:TEST-POINT3X4
- added U5: ESD Diode, SparkFun-DiscreteSemi:TVS_DIODE_ARRAY_DT1042-04SO-7
- added U7: AP63203, SparkFun-IC-Power:AP63203
- C4: value 1nF -> 0.1uF; device SparkFun-Capacitors:1.0NF/1000PF-0603-50V-10% -> SparkFun-Capacitors:0.1UF-0603-25V-10%-X7R-WE
- R17, R4: value 10k -> 100k; device SparkFun-Resistors:10KOHM-0603-1/10W-1% -> SparkFun-Resistors:100KOHM-0603-1/10W-1%
- R20: value 2.0k -> 1.5k; device SparkFun-Resistors:2.0KOHM-0603-1/10W-5% -> SparkFun-Resistors:1.5KOHM-0603-1/10W-1%
- U4: value CH340E_MSOP10 -> CH340C; device SparkFun-IC-Comms:CH340E_MSOP10 -> SparkFun-IC-Comms:CH340C
Connections:
- net ESP_23 renamed ESP_23/PICO
- removed net N$24: S.2, U1.VIO/!STDBY!
- removed net RESET: C4.1, R17.1, S1.2, U3.EN
- new net !RESET: Q2G1.E, R16.1, S2.2, U3.EN
- new net !STDBY: S.2, TP10.1, U1.VIO/!STDBY!
- new net 3.3V_LDO: C10.1, C11.1, C3.1, C4.1, D2.VCC, J7.2, L2.2, R16.2, U2G2.P$V+, U3.3V3, U7.FB
- new net DTR: Q2G2.E, R2.2, U4.!DTR
- new net EN: R17.1, U3.IO16, U6.EN
- new net ESP_0/QPWR: Q2G2.C, S1.2, TP1.1, U3.IOA0
- new net ESP_19/POCI: U3.POCI3/IO19
- new net ESP_21/TP_SDA: J7.3, U3.SDA/IO21
- new net ESP_22/TP_SCL: J7.4, U3.SCL/IO22
- new net ESP_34/AUX1: S4.1, U3.IA34
- new net ESP_35/AUX2: S3.1, U3.IA35
- new net N$10: C9.1, U7.BST
- new net N$12: D2.DO, TP2.1
- new net N$13: C11.2
- new net N$2: R22.1, R23.2, U7.EN
- new net N$7: Q2G1.B, R2.1
- new net N$8: Q2G2.B, R3.1
- new net N$9: C9.2, L2.1, U7.SW
- new net RTS: Q2G1.C, R3.2, U4.!RTS
- net 3.3V: no longer C3.1, R17.2, R4.2, U2G2.P$V+, U3.3V3
- net CURR_SENSE: now also R21.2, TP11.1; no longer R25.2
- net D+: now also U5.IO4
- net D-: now also U5.IO3
- net DIAG: now also TP9.1
- net ESP_0: no longer U3.IOA0
- net ESP_16: no longer U3.IO16
- net ESP_19: no longer U3.POCI3/IO19
- net ESP_21: no longer U3.SDA/IO21
- net ESP_22: no longer U3.SCL/IO22
- net ESP_34: now also D2.DI; no longer U3.IA34
- net ESP_35: no longer U3.IA35
- net GND: now also C10.2, C12.2, D2.GND, J7.1, J8.1, R23.1, S2.1, S3.2, S4.2, U5.VSS, U7.GND
- net N$28: now also D4.C; no longer D4.A
- net N$29: now also D4.A; no longer D4.C
- net N$6: now also R21.1; no longer R25.1
- net UH: now also TP3.1
- net UL: now also TP4.1
- net VH: now also TP5.1
- net VIN: now also C12.1, J8.2, R17.2, R22.2, R4.2, U7.VIN; no longer U6.EN
- net VL: now also TP6.1
- net V_USB: now also U5.VCC
- net WH: now also TP7.1
- net WL: now also TP8.1
Other:
- note added: "0"
- note added: "1"
- note added: "3-Pin Molex connector that mates nicely with this motor from SFE: ROB-20441"
- note added: "4.7uH"
- note added: "ADC2 is unavailable when WiFi is enabled."
- note added: "Auto-Reset"
- note added: "Auxilary Push Buttons: Use for any general purpose"
- note added: "Boot Mode Configuration"
- note added: "Bootloader"
- note added: "Breakout Headers"
- note added: "Breakout headers for use case of user choosing a different power connection other than USB or Power Jack"
- note added: "Cut SHLD jumper to disconnect USB Shield from GND"
- note added: "Default"
- note added: "GPIO0 and Reset Buttons"
- note added: "IO0"
- note added: "IO0: Avoid device connections. Can be used a stat LED."
- note added: "IO12"
- note added: "IO12 = MDTI, IO15 = MDTO"
- note added: "IO12: Avoid external pullups - will cause bootloader fail."
- note added: "IO15"
- note added: "IO15: Has builtin pullup at POR."
- note added: "IO2"
- note added: "IO2: Avoid external pullups - will cause bootloader fail."
- note added: "IO5"
- note added: "IO5: Has builtin pullup at POR."
- note added: "If DTR is LOW, toggling RTS from HIGH to LOW resets to run mode. If RTS is HIGH, toggling DTR from LOW to HIGH resets to bootloader."
- note added: "Isolated Power Supply"
- note added: "Pin"
- note added: "Qwiic Connector"
- note added: "RGB Status LED"
- note added: "Run"
- note added: "This is the penny-in-the-fuse jumper. Close only if you know what you're doing."
- note added: "Use boot control pins with caution: 0, 2, 5, 12, 15"
- note added: "WS2812"
- note added: "x"
- note removed: "Pin Headers"
- note removed: "Power LED"
- note removed: "RESET"
- note removed: "Reset"
- moved on the sheet: BYP, C1, C18, C19, C2, C20, C21, C3, C5, C6, C7, C8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
